File: MCU_Datalogger.kicad_sch (KiCad schematic)
At the start: 25 parts, among them U1 24LC1025, U2 24LC1025, U3 DS1337S_, U4 ATMEGA328P-AU, Y1 32.768 KHz, Y2 16 MHz

Commit message: sheet 1 wiring done
Connections:
- net GND: now also BT1.2 (-), C1.2, C2.1, C3.1, C4.1, C5.2, R5.1, R7.2, U1.4 (GND), U1.7 (WP), U2.2 (A1), U2.4 (GND), U2.7 (WP), U3.4 (GND)
- net at D1.1 (K): now also R7.1
- net at D1.2 (A): now also BT1.1 (+), C5.1, U4.18 (AVCC), U4.4 (VCC)
- net at C4.2: now also U4.20 (AREF)
- net at R5.2: now also D2.1 (K)
- net at C2.2: now also U4.7 (PB6), Y2.1
- net Vcc: now reaches R2.1
- net Vcc: now also C1.1, R1.2, R3.1, R4.1, R6.1, U1.1 (A0), U1.2 (A1), U1.3 (A2), U1.8 (VCC), U2.1 (A0), U2.3 (A2), U2.8 (VCC), U3.8 (VCC)
- net at R2.2: now also U3.7 (SQW/~INT)
- net at Y2.2: now also C3.2, U4.8 (PB7)
- net SCK: now reaches D2.2 (A)
- net SCK: now also R3.2, U1.6 (SCL), U2.6 (SCL), U3.6 (SCL), U4.17 (PB5), U4.28 (PC5)
- net SDA: now reaches R4.2
- net SDA: now also U1.5 (SDA), U2.5 (SDA), U3.5 (SDA), U4.27 (PC4)
- net RESET: now reaches R6.2
- net RESET: now also U4.29 (PC6/~{RESET})
- net at R1.1: now also U3.3 (~{INTA})
- net at Y1.1: now also U3.2 (X2)
- net at Y1.2: now also U3.1 (X1)
- net D3: now reaches U4.1 (PD3)
- net D6: now reaches U4.10 (PD6)
- net D7: now reaches U4.11 (PD7)
- net D8: now reaches U4.12 (PB0)
- net MOSI: now reaches U4.15 (PB3)
- net MISO: now reaches U4.16 (PB4)
- net D4: now reaches U4.2 (PD4)
- net RX: now reaches U4.30 (PD0)
- net TX: now reaches U4.31 (PD1)
- net D2: now reaches U4.32 (PD2)
- net D5: now reaches U4.9 (PD5)
- net VCC: no longer names the net of U4.6 (VCC)
- net VCC: no longer U4.4 (VCC)
- no-connect marks 0 -> 9
Other:
- moved on the sheet: BT1, C1, C2, C3, C4, C5, D1, D2, R1, R2, R4, R5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

Commit message: wiring in 2nd sheet done
Other:
- sheet Connectors ports: added D2, D3, D4, D5, D6, D7, D8, GND, MISO, MOSI, RESET, RX, SCK, SDA, TX, Vcc; removed none

Commit message: commits completed
Other:
- note added: "EEPROM"
- note added: "MCU"
- note added: "Mounting"
- note added: "Real Time Clock"
Changed lines of the file:
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@@
 		(rev "1")
+	)
+	(rectangle
+		(start 35.56 121.285)
+		(end 142.24 166.37)
+		(stroke
+			(width 0)
+			(type dash)
+		)
+		(fill
+			(type none)
+		)
+	)
+	(rectangle
+		(start 256.54 127)
+		(end 280.035 158.115)
+		(stroke
+			(width 0)
+			(type dash)
+		)
+		(fill
+			(type none)
+		)
+	)
+	(rectangle
+		(start 24.765 26.035)
+		(end 132.08 86.36)
+		(stroke
+			(width 0)
+			(type dash)
+		)
+		(fill
+			(type none)
+		)
+	)
+	(rectangle
+		(start 137.16 19.685)
+		(end 284.48 98.425)
+		(stroke
+			(width 0)
+			(type dash)
+		)
+		(fill
+			(type none)
+		)
+	)
+	(text "EEPROM"
+		(exclude_from_sim no)
+		(at 39.37 119.38 0)
+		(effects
+			(font
+				(size 1.27 1.27)
+				(thickness 0.254)
+				(bold yes)
+			)
+		)
+	)
+	(text "MCU\n"
+		(exclude_from_sim no)
+		(at 139.7 19.05 0)
+		(effects
+			(font
+				(size 1.27 1.27)
+				(thickness 0.254)
+				(bold yes)
+			)
+		)
+	)
+	(text "Mounting"
+		(exclude_from_sim no)
+		(at 260.35 125.73 0)
+		(effects
+			(font
+				(size 1.27 1.27)
+				(thickness 0.254)
+				(bold yes)
+			)
+		)
+	)
+	(text "Real Time Clock"
+		(exclude_from_sim no)
+		(at 33.02 25.4 0)
+		(effects
+			(font
+				(size 1.27 1.27)
+				(thickness 0.254)
+				(bold yes)
+			)
+		)
 	)
 	(junction
