File: .history/MCU_Datalogger.kicad_sch (KiCad schematic)
At the start: 25 parts, among them U1 24LC1025, U2 24LC1025, U3 DS1337S_, U4 ATMEGA328P-AU, Y1 32.768 KHz, Y2 16 MHz

Commit message: setup PCB new
Other:
- note added: "Mounting"
Changed lines of the file:
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@@
+		)
+	)
+	(text "Mounting"
+		(exclude_from_sim no)
+		(at 260.35 125.73 0)
+		(effects
+			(font
+				(size 1.27 1.27)
+				(thickness 0.254)
+				(bold yes)
+			)
 		)
 	)
