File: .history/MCU_Datalogger.kicad_sch (KiCad schematic)
At the start: 25 parts, among them U1 24LC1025, U2 24LC1025, U3 DS1337S_, U4 ATMEGA328P-AU, Y1 32.768 KHz, Y2 16 MHz

Commit message: footprint assigned
Parts:
- BT1: footprint (none) -> Connector_PinHeader_2.54mm:PinHeader_1x02_P2.54mm_Vertical
- C1, C2, C3, C4, C5: footprint (none) -> Capacitor_SMD:C_0805_2012Metric
- D1, D2: footprint (none) -> LED_SMD:LED_0805_2012Metric
- H1, H2, H3, H4: footprint (none) -> MountingHole:MountingHole_2.1mm
- R1, R2, R3, R4, R5, R6, R7: footprint (none) -> Resistor_SMD:R_0805_2012Metric
- U1, U2: footprint (none) -> Package_SO:SOIC-8_5.3x5.3mm_P1.27mm
- U3: footprint DS1337S_:SOIC127P600X175-8N -> Footprints:SOIC127P600X175-8N
- U4: footprint ATMEGA328P-AU:QFP80P900X900X120-32N -> Footprints:QFP80P900X900X120-32N
- Y1, Y2: footprint (none) -> Crystal:Crystal_SMD_5032-2Pin_5.0x3.2mm_HandSoldering
Changed lines of the file:
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@@
 			)
 		)
-		(property "Footprint" ""
+		(property "Footprint" "LED_SMD:LED_0805_2012Metric"
 			(at 247.65 50.8 0)
 			(hide yes)
@@
 			)
 		)
-		(property "Footprint" ""
+		(property "Footprint" "Capacitor_SMD:C_0805_2012Metric"
 			(at 186.69 26.9748 0)
 			(hide yes)
@@
 			)
 		)
-		(property "Footprint" ""
+		(property "Footprint" "Connector_PinHeader_2.54mm:PinHeader_1x02_P2.54mm_Vertical"
 			(at 261.62 31.496 90)
 			(hide yes)
@@
 			)
 		)
-		(property "Footprint" ""
+		(property "Footprint" "Resistor_SMD:R_0805_2012Metric"
 			(at 167.64 42.418 90)
 			(hide yes)
@@
 			)
 		)
-		(property "Footprint" ""
+		(property "Footprint" "MountingHole:MountingHole_2.1mm"
 			(at 261.62 144.78 0)
 			(hide yes)
@@
 			)
 		)
-		(property "Footprint" ""
+		(property "Footprint" "Capacitor_SMD:C_0805_2012Metric"
 			(at 169.8752 58.42 0)
 			(hide yes)
@@
 			)
 		)
-		(property "Footprint" ""
+		(property "Footprint" "Resistor_SMD:R_0805_2012Metric"
 			(at 106.172 43.18 90)
 			(hide yes)
@@
 			)
 		)
-		(property "Footprint" ""
+		(property "Footprint" "Crystal:Crystal_SMD_5032-2Pin_5.0x3.2mm_HandSoldering"
 			(at 184.15 60.96 0)
 			(hide yes)
@@
 			)
 		)
-		(property "Footprint" ""
+		(property "Footprint" "Resistor_SMD:R_0805_2012Metric"
 			(at 245.872 62.23 90)
 			(hide yes)
@@
 			)
 		)
-		(property "Footprint" ""
+		(property "Footprint" "Capacitor_SMD:C_0805_2012Metric"
 			(at 242.2652 36.83 0)
 			(hide yes)
@@
 			)
 		)
-		(property "Footprint" ""
+		(property "Footprint" "MountingHole:MountingHole_2.1mm"
 			(at 261.62 132.08 0)
 			(hide yes)
@@
 			)
 		)
-		(property "Footprint" ""
+		(property "Footprint" "LED_SMD:LED_0805_2012Metric"
 			(at 185.42 41.91 0)
 			(hide yes)
@@
 			)
 		)
-		(property "Footprint" ""
+		(property "Footprint" "Resistor_SMD:R_0805_2012Metric"
 			(at 122.682 146.05 90)
 			(hide yes)
@@
 			)
 		)
-		(property "Footprint" ""
+		(property "Footprint" "Resistor_SMD:R_0805_2012Metric"
 			(at 184.15 84.328 90)
 			(hide yes)
@@
 			)
 		)
-		(property "Footprint" ""
+		(property "Footprint" "MountingHole:MountingHole_2.1mm"
 			(at 261.62 151.13 0)
 			(hide yes)
@@
 			)
 		)
-		(property "Footprint" ""
+		(property "Footprint" "MountingHole:MountingHole_2.1mm"
 			(at 261.62 138.43 0)
 			(hide yes)
@@
 			)
 		)
-		(property "Footprint" ""
+		(property "Footprint" "Resistor_SMD:R_0805_2012Metric"
 			(at 113.792 146.05 90)
 			(hide yes)
@@
 			)
 		)
-		(property "Footprint" ""
+		(property "Footprint" "Resistor_SMD:R_0805_2012Metric"
 			(at 99.568 43.18 90)
 			(hide yes)
@@
 			)
 		)
-		(property "Footprint" ""
+		(property "Footprint" "Crystal:Crystal_SMD_5032-2Pin_5.0x3.2mm_HandSoldering"
 			(at 39.37 57.15 0)
 			(hide yes)
@@
 			)
 		)
-		(property "Footprint" ""
+		(property "Footprint" "Package_SO:SOIC-8_5.3x5.3mm_P1.27mm"
 			(at 86.36 146.05 0)
 			(hide yes)
@@
 			)
 		)
-		(property "Footprint" "ATMEGA328P-AU:QFP80P900X900X120-32N"
+		(property "Footprint" "Footprints:QFP80P900X900X120-32N"
 			(at 217.17 62.23 0)
 			(hide yes)
@@
 			)
 		)
-		(property "Footprint" "DS1337S_:SOIC127P600X175-8N"
+		(property "Footprint" "Footprints:SOIC127P600X175-8N"
 			(at 69.85 57.15 0)
 			(hide yes)
@@
 			)
 		)
-		(property "Footprint" ""
+		(property "Footprint" "Capacitor_SMD:C_0805_2012Metric"
 			(at 171.1452 74.93 0)
 			(hide yes)
@@
 			)
 		)
-		(property "Footprint" ""
+		(property "Footprint" "Package_SO:SOIC-8_5.3x5.3mm_P1.27mm"
 			(at 59.69 146.05 0)
 			(hide yes)
@@
 			)
 		)
-		(property "Footprint" ""
+		(property "Footprint" "Capacitor_SMD:C_0805_2012Metric"
 			(at 122.8852 46.99 0)
 			(hide yes)

Commit message: sheet 1 wiring done
Connections:
- net GND: now also BT1.2 (-), C1.2, C2.1, C3.1, C4.1, C5.2, R5.1, R7.2, U1.4 (GND), U1.7 (WP), U2.2 (A1), U2.4 (GND), U2.7 (WP), U3.4 (GND)
- net at D1.1 (K): now also R7.1
- net at D1.2 (A): now also BT1.1 (+), C5.1, U4.18 (AVCC), U4.4 (VCC)
- net at C4.2: now also U4.20 (AREF)
- net at R5.2: now also D2.1 (K)
- net at C2.2: now also U4.7 (PB6), Y2.1
- net Vcc: now reaches R2.1
- net Vcc: now also C1.1, R1.2, R3.1, R4.1, R6.1, U1.1 (A0), U1.2 (A1), U1.3 (A2), U1.8 (VCC), U2.1 (A0), U2.3 (A2), U2.8 (VCC), U3.8 (VCC)
- net at R2.2: now also U3.7 (SQW/~INT)
- net at Y2.2: now also C3.2, U4.8 (PB7)
- net SCK: now reaches D2.2 (A)
- net SCK: now also R3.2, U1.6 (SCL), U2.6 (SCL), U3.6 (SCL), U4.17 (PB5), U4.28 (PC5)
- net SDA: now reaches R4.2
- net SDA: now also U1.5 (SDA), U2.5 (SDA), U3.5 (SDA), U4.27 (PC4)
- net RESET: now reaches R6.2
- net RESET: now also U4.29 (PC6/~{RESET})
- net at R1.1: now also U3.3 (~{INTA})
- net at Y1.1: now also U3.2 (X2)
- net at Y1.2: now also U3.1 (X1)
- net D3: now reaches U4.1 (PD3)
- net D6: now reaches U4.10 (PD6)
- net D7: now reaches U4.11 (PD7)
- net D8: now reaches U4.12 (PB0)
- net MOSI: now reaches U4.15 (PB3)
- net MISO: now reaches U4.16 (PB4)
- net D4: now reaches U4.2 (PD4)
- net RX: now reaches U4.30 (PD0)
- net TX: now reaches U4.31 (PD1)
- net D2: now reaches U4.32 (PD2)
- net D5: now reaches U4.9 (PD5)
- net VCC: no longer names the net of U4.6 (VCC)
- net VCC: no longer U4.4 (VCC)
- no-connect marks 0 -> 7
Other:
- moved on the sheet: BT1, C1, C2, C3, C4, C5, D1, D2, R1, R2, R4, R5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

Commit message: wiring in 2nd sheet done
Connections:
- no-connect marks 7 -> 9
Other:
- sheet Connectors ports: added D2, D3, D4, D5, D6, D7, D8, GND, MISO, MOSI, RESET, RX, SCK, SDA, TX, Vcc; removed none

Commit message: commits completed
Other:
- note added: "EEPROM"
- note added: "MCU"
- note added: "Real Time Clock"
Changed lines of the file:
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@@
 		(rev "1")
+	)
+	(rectangle
+		(start 35.56 121.285)
+		(end 142.24 166.37)
+		(stroke
+			(width 0)
+			(type dash)
+		)
+		(fill
+			(type none)
+		)
+	)
+	(rectangle
+		(start 256.54 127)
+		(end 280.035 158.115)
+		(stroke
+			(width 0)
+			(type dash)
+		)
+		(fill
+			(type none)
+		)
+	)
+	(rectangle
+		(start 24.765 26.035)
+		(end 132.08 86.36)
+		(stroke
+			(width 0)
+			(type dash)
+		)
+		(fill
+			(type none)
+		)
+	)
+	(rectangle
+		(start 137.16 19.685)
+		(end 284.48 98.425)
+		(stroke
+			(width 0)
+			(type dash)
+		)
+		(fill
+			(type none)
+		)
+	)
+	(text "EEPROM"
+		(exclude_from_sim no)
+		(at 39.37 119.38 0)
+		(effects
+			(font
+				(size 1.27 1.27)
+				(thickness 0.254)
+				(bold yes)
+			)
+		)
+	)
+	(text "MCU\n"
+		(exclude_from_sim no)
+		(at 139.7 19.05 0)
+		(effects
+			(font
+				(size 1.27 1.27)
+				(thickness 0.254)
+				(bold yes)
+			)
+		)
+	)
+	(text "Real Time Clock"
+		(exclude_from_sim no)
+		(at 33.02 25.4 0)
+		(effects
+			(font
+				(size 1.27 1.27)
+				(thickness 0.254)
+				(bold yes)
+			)
+		)
 	)
 	(junction

Commit message: starting 4 layer PCB
Connections:
- net Vcc: now also BT1.1 (+), C5.1, D1.2 (A), U4.18 (AVCC), U4.4 (VCC)
Other:
- note added: "Mounting"
Changed lines of the file:
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@@
+		)
+	)
+	(text "Mounting"
+		(exclude_from_sim no)
+		(at 260.35 125.73 0)
+		(effects
+			(font
+				(size 1.27 1.27)
+				(thickness 0.254)
+				(bold yes)
+			)
 		)
 	)
@@
 		(effects
 			(font
+				(size 1.27 1.27)
+			)
+			(justify left bottom)
+		)
+	)
+	(label "Vcc"
+		(at 265.43 36.83 0)
+		(effects
+			(font

Commit message: 4 layer pcb done
Connections:
- net Vcc: no longer BT1.1 (+), C5.1, D1.2 (A), U4.18 (AVCC), U4.4 (VCC)
- new net: BT1.1 (+), C5.1, D1.2 (A), U4.18 (AVCC), U4.4 (VCC)
Changed lines of the file:
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@@
-		)
-	)
-	(label "Vcc"
-		(at 265.43 36.83 0)
-		(effects
-			(font
-				(size 1.27 1.27)
-			)
-			(justify left bottom)
 		)
 	)

Commit message: all done board
Connections:
- net Vcc: now also BT1.1 (+), C5.1, D1.2 (A), U4.18 (AVCC), U4.4 (VCC)
Changed lines of the file:
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@@
+		)
+	)
+	(label "Vcc"
+		(at 265.43 36.83 0)
+		(effects
+			(font
+				(size 1.27 1.27)
+			)
+			(justify left bottom)
 		)
 	)
