File: .history/MCU_Datalogger.kicad_pcb (KiCad board)
At the start: 2 copper layers, 29 parts, among them J1 Conn_01x04_Pin, J2 Conn_01x04_Pin, J3 Conn_01x09_Pin, J4 Conn_02x03_Odd_Even, U1 24LC1025, U2 24LC1025, U3 DS1337S_, U4 ATMEGA328P-AU, Y1 32.768 KHz, Y2 16 MHz

Commit message: footprint placement completed
Parts:
- moved H2 44.0 mm to (156.2, 64.1)
- moved H4 43.3 mm to (156.2, 93.3)
- moved J3 38.7 mm to (115.6, 92.1), turned to 90 degrees
- moved R5 30.5 mm to (147.0, 68.6)
- moved R6 30.4 mm to (147.0, 71.8)
- moved Y1 29.0 mm to (111.1, 83.1), turned to 90 degrees
- moved R7 28.3 mm to (141.3, 68.6)
- moved J2 27.0 mm to (142.2, 92.1), turned to 90 degrees
- moved C5 27.0 mm to (136.2, 66.7)
- moved H1 24.6 mm to (109.9, 93.3)
- moved R4 23.2 mm to (141.3, 71.8)
- moved R3 22.8 mm to (141.3, 74.9)
- moved C3 21.2 mm to (131.8, 66.7)
- moved R1 20.1 mm to (116.6, 87.6)
- moved D2 19.3 mm to (141.3, 65.4)
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Other:
- board outline added: 51.7 x 34.5 mm

Commit message: routing done, fill is pending
Parts:
- moved U2 8.25 mm to (118.7, 67.3)
- moved U1 6.99 mm to (118.7, 74.9)
- moved D1 5.72 mm to (141.3, 65.4)
- moved D2 5.72 mm to (147.0, 65.4)
- moved BT1 2.54 mm to (111.1, 71.1), turned to 0 degrees
- turned R1 to 180 degrees
- turned R2 to 180 degrees
- turned R3 to 180 degrees
- turned R4 to 180 degrees
- turned R5 to 180 degrees
Routing:
- net /Vcc: track 0.00 -> 145.8 mm, vias 0 -> 1
- net /SCK: track 0.00 -> 94.5 mm, vias 0 -> 4
- net /SDA: track 0.00 -> 66.3 mm, vias 0 -> 5
- net GND: track 0.00 -> 57.1 mm, vias 0 -> 6
- net Net-(BT1-+): track 0.00 -> 56.0 mm, vias 0 -> 6
- net /MOSI: track 0.00 -> 38.1 mm, vias 0 -> 1
- net /TX: track 0.00 -> 31.8 mm, vias 0 -> 1
- net Net-(U4-PB6): track 0.00 -> 30.7 mm
- net Net-(U4-PB7): track 0.00 -> 29.9 mm, vias 0 -> 4
- net /RX: track 0.00 -> 29.8 mm, vias 0 -> 1
- net /D2: track 0.00 -> 28.9 mm, vias 0 -> 1
- net /RESET: track 0.00 -> 26.6 mm, vias 0 -> 2
- net /MISO: track 0.00 -> 25.0 mm
- net /D3: track 0.00 -> 23.9 mm, vias 0 -> 1
- net /D4: track 0.00 -> 21.6 mm, vias 0 -> 1
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
Commit message: routing completed
Routing:
- net GND: track 57.1 -> 119.3 mm, vias 6 -> 14
- net /Vcc: track 145.8 -> 121.0 mm
- net /MOSI: track 38.1 -> 42.7 mm
- net Net-(BT1-+): track 56.0 -> 58.3 mm
- net /RESET: track 26.6 -> 27.9 mm
- net /D4: track 21.6 -> 22.1 mm
- added copper zone on F.Cu, net /Vcc
- added copper zone on B.Cu, net GND

Commit message: routing fixes
Routing:
- net /Vcc: track 121.0 -> 129.4 mm, vias 1 -> 5
Changed lines of the file:
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@@
 		(tags "mountinghole")
 		(property "Reference" "H3"
-			(at 0 -3.05 0)
+			(at 3.1242 -1.7526 0)
 			(layer "F.SilkS")
 			(effects
@@
 		(tags "resistor")
 		(property "Reference" "R7"
-			(at 0 -1.65 0)
+			(at -1.4751 -1.524 0)
 			(layer "F.SilkS")
 			(effects
@@
 		(tags "resistor")
 		(property "Reference" "R6"
-			(at 0 -1.65 0)
+			(at 2.6143 0.0762 0)
 			(layer "F.SilkS")
 			(effects
@@
 		(tags "mountinghole")
 		(property "Reference" "H2"
-			(at 0 -3.05 0)
+			(at -2.9972 -1.8542 0)
 			(layer "F.SilkS")
 			(effects
@@
 	)
 	(segment
+		(start 115.65 87.63)
+		(end 115.65 86.694)
+		(width 0.2)
+		(layer "F.Cu")
+		(net "/Vcc")
+	)
+	(segment
 		(start 142.24 73.152)
 		(end 142.24 71.755)
@@
 	)
 	(segment
+		(start 115.65 86.694)
+		(end 115.1128 86.1568)
+		(width 0.2)
+		(layer "F.Cu")
+		(net "/Vcc")
+	)
+	(segment
 		(start 118.872 85.217)
 		(end 118.872 82.804)
@@
 		(net "/Vcc")
 	)
+	(via
+		(at 113.2332 89.7636)
+		(size 0.6)
+		(drill 0.3)
+		(layers "F.Cu" "B.Cu")
+		(net "/Vcc")
+	)
+	(via
+		(at 150.8252 65.3288)
+		(size 0.6)
+		(drill 0.3)
+		(layers "F.Cu" "B.Cu")
+		(net "/Vcc")
+	)
+	(via
+		(at 150.622 63.0428)
+		(size 0.6)
+		(drill 0.3)
+		(layers "F.Cu" "B.Cu")
+		(net "/Vcc")
+	)
+	(via
+		(at 115.1128 86.1568)
+		(size 0.6)
+		(drill 0.3)
+		(layers "F.Cu" "B.Cu")
+		(net "/Vcc")
+	)
 	(segment
 		(start 157.226 88.392)
@@
 	)
 	(segment
+		(start 115.1128 86.1568)
+		(end 113.2332 88.0364)
+		(width 0.2)
+		(layer "B.Cu")
+		(net "/Vcc")
+	)
+	(segment
 		(start 156.591 81.915)
 		(end 154.94 81.915)
@@
 	)
 	(segment
+		(start 150.8252 63.246)
+		(end 150.622 63.0428)
+		(width 0.2)
+		(layer "B.Cu")
+		(net "/Vcc")
+	)
+	(segment
 		(start 152.781 67.056)
 		(end 154.94 69.215)
@@
 	)
 	(segment
+		(start 113.2332 88.0364)
+		(end 113.2332 89.7636)
+		(width 0.2)
+		(layer "B.Cu")
+		(net "/Vcc")
+	)
+	(segment
 		(start 151.384 94.234)
 		(end 157.226 88.392)
@@
 		(width 0.2)
 		(layer "B.Cu")
+		(net "/Vcc")
+	)
+	(segment
+		(start 150.8252 65.3288)
+		(end 150.8252 63.246)
+		(width 0.2)
+		(layer "B.Cu")

Commit message: all done board
Connections:
- BT1 pad 1: Net-(BT1-+) -> /Vcc
- C5 pad 1: Net-(BT1-+) -> /Vcc
- D1 pad 2: Net-(BT1-+) -> /Vcc
- U4 pad 18: Net-(BT1-+) -> /Vcc
- U4 pad 4: Net-(BT1-+) -> /Vcc
Routing:
- net Net-(BT1-+): track 58.3 -> 0.00 mm, vias 6 -> 0
- net /Vcc: track 129.4 -> 187.7 mm, vias 5 -> 11
Other:
- board text added: "2"
- board text added: "3"
- board text added: "4"
- board text added: "5"
- board text added: "6"
- board text added: "7"
- board text added: "8"
- board text added: "Data Logger with the ATMega328P - 2Mbit EEPROM - RTC - I2C, SPI, GPIOs"
- board text added: "GND"
- board text added: "I2C"
- board text added: "ICSP"
- board text added: "ICSP MOSI | Vcc SCK | MISO RESET| GND"
- board text added: "RX"
- board text added: "SCK"
- board text added: "SDA"
- board text added: "SERIAL"
- board text added: "TX"
- board text added: "Vcc"
