File: .history/MCU_Datalogger.kicad_pcb (KiCad board)
At the start: 4 copper layers, 51.7 x 34.5 mm, 29 parts, among them J1 Conn_01x04_Pin, J2 Conn_01x04_Pin, J3 Conn_01x09_Pin, J4 Conn_02x03_Odd_Even, U1 24LC1025, U2 24LC1025, U3 DS1337S_, U4 ATMEGA328P-AU, Y1 32.768 KHz, Y2 16 MHz

Commit message: 4 layer pcb done
Parts:
- moved Y2 0.90 mm to (132.7, 85.7)
Routing:
- net /SCK: track 0.00 -> 90.7 mm, vias 0 -> 7
- net /SDA: track 0.00 -> 62.9 mm, vias 0 -> 6
- net GND: track 0.00 -> 44.1 mm, vias 0 -> 12
- net /Vcc: track 0.00 -> 40.4 mm, vias 0 -> 13
- net /TX: track 0.00 -> 40.3 mm
- net /RX: track 0.00 -> 36.6 mm
- net Net-(U4-PB6): track 0.00 -> 36.2 mm, vias 0 -> 4
- net /D2: track 0.00 -> 30.6 mm
- net /MISO: track 0.00 -> 30.0 mm, vias 0 -> 2
- net /MOSI: track 0.00 -> 29.2 mm, vias 0 -> 2
- net Net-(U4-PB7): track 0.00 -> 28.5 mm, vias 0 -> 3
- net /RESET: track 0.00 -> 24.8 mm, vias 0 -> 2
- net /D3: track 0.00 -> 24.6 mm
- net /D4: track 0.00 -> 22.0 mm
- net /D8: track 0.00 -> 16.4 mm
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- added copper zone on In2.Cu, net /Vcc
- added copper zone on B.Cu, net GND
